File: motor_controller/motor_controller.kicad_pcb (KiCad board)
At the start: 2 copper layers, 69.1 x 53.8 mm, 25 parts, among them J101 Conn_01x06, J102 Conn_01x06, J103 Barrel_Jack_Switch, J104 Conn_01x06, J105 Conn_01x08, J106 Conn_01x06, J107 Conn_01x10, J108 Conn_01x08, U101 MAX14780, U102 MAX14780

Commit message: updated schematic pdf and generated gerber files
Other:
- board text added: "Alan Ford Rev. 0 - 1/20/2020"
- board text removed: "Alan Ford Rev. 0 - 1/11/2020"
Changed lines of the file:
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@@
     (pcbplotparams
       (layerselection 0x010fc_ffffffff)
-      (usegerberextensions false)
+      (usegerberextensions true)
       (usegerberattributes false)
       (usegerberadvancedattributes false)
@@
       (psnegative false)
       (psa4output false)
-      (plotreference true)
-      (plotvalue true)
+      (plotreference false)
+      (plotvalue false)
       (plotinvisibletext false)
       (padsonsilk false)
@@
       (outputformat 1)
       (mirror false)
-      (drillshape 1)
+      (drillshape 0)
       (scaleselection 1)
-      (outputdirectory ""))
+      (outputdirectory "gerbers/"))
   )
   (net 0 "")
@@
     (effects (font (size 1.5 1.5) (thickness 0.3)))
   )
-  (gr_text "Alan Ford\nRev. 0 - 1/11/2020" (at 178.435 88.265) (layer B.SilkS)
+  (gr_text "Alan Ford\nRev. 0 - 1/20/2020" (at 178.435 88.265) (layer B.SilkS)
     (effects (font (size 1.5 1.5) (thickness 0.3)) (justify left mirror))
   )
